File: Encoder_check.kicad_pcb (KiCad board)
At the start: 2 copper layers, 64 x 71 mm, 92 parts, among them J1 Conn_01x10, J2 Conn_01x06, J3 Conn_01x04, J4 Screw_Terminal_01x06, J5 Conn_01x02, J6 Screw_Terminal_01x02, J7 Barrel_Jack_Switch, J8 Screw_Terminal_01x02, J9 Screw_Terminal_01x04, P1 Digital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

Commit message: SPIにつなぐデバイスの電圧が違ったため設計ミスが判明。 これを修正した
Parts:
- removed RN4, RN5, RN6: R_Pack02, Resistor_SMD:R_Array_Concave_2x0603
- added R29: 10k, Resistor_SMD:R_0603_1608Metric, F.Cu at (182.6, 104.5)
- added R30: 20k, Resistor_SMD:R_0603_1608Metric, F.Cu at (181.0, 104.5)
- added R31: 10k, Resistor_SMD:R_0603_1608Metric, F.Cu at (182.6, 99.5)
- added R32: 20k, Resistor_SMD:R_0603_1608Metric, F.Cu at (181.0, 99.5)
- added R33: 10k, Resistor_SMD:R_0603_1608Metric, F.Cu at (182.6, 94.5)
- added R34: 20k, Resistor_SMD:R_0603_1608Metric, F.Cu at (181.0, 94.5)
- J1: value Conn_01x10 -> Conn_02x05_Odd_Even
- J2: value Conn_01x06 -> Screw_Terminal_01x06
- RN1, RN2, RN3: value R_Pack02 -> 150
- moved C4 1.44 mm to (181.1, 75.7), turned to 90 degrees
Connections:
- C4 pad 1: +5V -> +3V3
- R17 pad 2: +5V -> +3V3
- U2 pad 13: +5V -> +3V3
- U2 pad 14: +5V -> +3V3
Routing:
- net +3V3: track 160.1 -> 177.2 mm, vias 5 -> 7
- net GND: track 371.0 -> 359.1 mm, vias 152 -> 151
- net +5V: track 223.2 -> 211.3 mm, vias 8 -> 7
- net (no net): vias 0 -> 1
