File: Encoder_check.sch (KiCad schematic (older format))
At the start: 36 parts, among them J1 Conn_01x10, J2 Conn_01x06, J3 Conn_01x04, J4 Screw_Terminal_01x06, J6 Screw_Terminal_01x02, J7 Barrel_Jack_Switch, J8 Screw_Terminal_01x02, J9 Screw_Terminal_01x04, P1 Digital, P2 Analog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

Commit message: SPIにつなぐデバイスの電圧が違ったため設計ミスが判明。 これを修正した
Parts:
- removed J1: Conn_01x10, Connector_Multicomp:Multicomp_MC9A12-1034_2x05_P2.54mm_Vertical, symbol Connector_Generic:Conn_01x10
- removed J2: Conn_01x06, TerminalBlock_TE-Connectivity:TerminalBlock_TE_282834-6_1x06_P2.54mm_Horizontal, symbol Connector_Generic:Conn_01x06
- added J1: Conn_02x05_Odd_Even, Connector_Multicomp:Multicomp_MC9A12-1034_2x05_P2.54mm_Vertical, symbol Connector_Generic:Conn_02x05_Odd_Even
- added J2: Screw_Terminal_01x06, TerminalBlock_TE-Connectivity:TerminalBlock_TE_282834-6_1x06_P2.54mm_Horizontal, symbol Connector:Screw_Terminal_01x06
- D11: value LED -> LED_RED
- R1, R2, R27, R28, R3: value R -> 1k
- R26: value R -> 10k
- TC1: symbol mylib:Thermocouple_PCB -> Encoder_check-rescue:Thermocouple_PCB-mylib
- U5: symbol mylib:M78AR05-1 -> Encoder_check-rescue:M78AR05-1-mylib
Connections:
- net +5V: now also J1.3 (Pin_3), J2.2 (Pin_2)
- net GND: now also J1.2 (Pin_2), J2.1 (Pin_1)
- net inc_encoder/A+: now also J1.5 (Pin_5)
- net inc_encoder/A-: now also J1.6 (Pin_6)
- net inc_encoder/B+: now also J1.7 (Pin_7)
- net inc_encoder/B-: now also J1.8 (Pin_8)
- net inc_encoder/I+: now also J1.9 (Pin_9)
- net inc_encoder/I-: now also J1.10 (Pin_10)
- net ssi_encoder/C_+: now also J2.4 (Pin_4)
- net ssi_encoder/C_-: now also J2.3 (Pin_3)
- net ssi_encoder/D_+: now also J2.6 (Pin_6)
- net ssi_encoder/D_-: now also J2.5 (Pin_5)
Other:
- moved on the sheet: J3
Changed lines of the file:
@@
 EESchema Schematic File Version 4
-LIBS:Encoder_check-cache
 EELAYER 30 0
 EELAYER END
@@
 P 1700 5700
 F 0 "R1" H 1770 5746 50  0000 L CNN
-F 1 "R" H 1770 5655 50  0000 L CNN
+F 1 "1k" H 1770 5655 50  0000 L CNN
 F 2 "Resistor_SMD:R_0603_1608Metric" V 1630 5700 50  0001 C CNN
 F 3 "~" H 1700 5700 50  0001 C CNN
@@
 P 2100 5700
 F 0 "R2" H 2170 5746 50  0000 L CNN
-F 1 "R" H 2170 5655 50  0000 L CNN
+F 1 "1k" H 2170 5655 50  0000 L CNN
 F 2 "Resistor_SMD:R_0603_1608Metric" V 2030 5700 50  0001 C CNN
 F 3 "~" H 2100 5700 50  0001 C CNN
@@
 P 2450 5700
 F 0 "R3" H 2520 5746 50  0000 L CNN
-F 1 "R" H 2520 5655 50  0000 L CNN
+F 1 "1k" H 2520 5655 50  0000 L CNN
 F 2 "Resistor_SMD:R_0603_1608Metric" V 2380 5700 50  0001 C CNN
 F 3 "~" H 2450 5700 50  0001 C CNN
@@
 L power:GND #PWR0101
 U 1 1 5E35CD0B
-P 4400 3600
+P 3400 3700
 AR Path="/5E35CD0B" Ref="#PWR0101"  Part="1"
 AR Path="/5E34E778/5E35CD0B" Ref="#PWR?"  Part="1"
-F 0 "#PWR0101" H 4400 3350 50  0001 C CNN
-F 1 "GND" H 4405 3427 50  0000 C CNN
-F 2 "" H 4400 3600 50  0001 C CNN
-F 3 "" H 4400 3600 50  0001 C CNN
-	1    4400 3600
-	1    0    0    -1
-$EndComp
-Wire Wire Line
-	4050 3650 4100 3650
-Wire Wire Line
-	4100 3650 4100 3550
-Wire Wire Line
-	4400 3550 4400 3600
-Wire Wire Line
-	4050 3750 4200 3750
-Wire Wire Line
-	4050 4250 4600 4250
-Wire Wire Line
-	4050 4150 4600 4150
-Wire Wire Line
-	4050 4050 4600 4050
-Wire Wire Line
-	4050 3950 4600 3950
-Wire Wire Line
-	4050 4350 4600 4350
-Wire Wire Line
-	4050 4450 4600 4450
+F 0 "#PWR0101" H 3400 3450 50  0001 C CNN
+F 1 "GND" H 3405 3527 50  0000 C CNN
+F 2 "" H 3400 3700 50  0001 C CNN
+F 3 "" H 3400 3700 50  0001 C CNN
+	1    3400 3700
+	1    0    0    -1
+$EndComp
+Wire Wire Line
+	3400 3650 3400 3700
 Wire Wire Line
 	6250 1650 6700 1650
@@
 5(**)
 $Sheet
-S 2150 3750 650  400
+S 1650 2850 650  400
 U 5E328173
 F0 "rs485" 50
 F1 "rs485.sch" 50
-F2 "RO" O R 2800 3850 50
-F3 "DE" I R 2800 3950 50
-F4 "DI" I R 2800 4050 50
-F5 "RS485_+" B L 2150 3900 50
-F6 "RS485_-" B L 2150 4000 50
+F2 "RO" O R 2300 2950 50
+F3 "DE" I R 2300 3050 50
+F4 "DI" I R 2300 3150 50
+F5 "RS485_+" B L 1650 3000 50
+F6 "RS485_-" B L 1650 3100 50
 $EndSheet
 $Comp
 L Connector_Generic:Conn_01x04 J3
 U 1 1 5E3300C4
-P 1500 3800
-F 0 "J3" H 1418 4117 50  0000 C CNN
-F 1 "Conn_01x04" H 1418 4026 50  0000 C CNN
-F 2 "Connector_JST:JST_EH_S4B-EH_1x04_P2.50mm_Horizontal" H 1500 3800 50  0001 C CNN
-F 3 "~" H 1500 3800 50  0001 C CNN
-	1    1500 3800
+P 1000 2900
+F 0 "J3" H 918 3217 50  0000 C CNN
+F 1 "Conn_01x04" H 918 3126 50  0000 C CNN
+F 2 "Connector_JST:JST_EH_S4B-EH_1x04_P2.50mm_Horizontal" H 1000 2900 50  0001 C CNN
+F 3 "~" H 1000 2900 50  0001 C CNN
+	1    1000 2900
 	-1   0    0    -1
 $EndComp
@@
 L power:+24V #PWR0132
 U 1 1 5E339197
-P 2000 3550
-F 0 "#PWR0132" H 2000 3400 50  0001 C CNN
-F 1 "+24V" H 2015 3723 50  0000 C CNN
-F 2 "" H 2000 3550 50  0001 C CNN
-F 3 "" H 2000 3550 50  0001 C CNN
-	1    2000 3550
-	1    0    0    -1
-$EndComp
-Wire Wire Line
-	1700 3800 2000 3800
-Wire Wire Line
-	2000 3800 2000 3550
+P 1500 2650
+F 0 "#PWR0132" H 1500 2500 50  0001 C CNN
+F 1 "+24V" H 1515 2823 50  0000 C CNN
+F 2 "" H 1500 2650 50  0001 C CNN
+F 3 "" H 1500 2650 50  0001 C CNN
+	1    1500 2650
+	1    0    0    -1
+$EndComp
+Wire Wire Line
+	1200 2900 1500 2900
+Wire Wire Line
+	1500 2900 1500 2650
 $Comp
 L power:GND #PWR0133
 U 1 1 5E33C53F
-P 1800 4100
-F 0 "#PWR0133" H 1800 3850 50  0001 C CNN
-F 1 "GND" H 1805 3927 50  0000 C CNN
-F 2 "" H 1800 4100 50  0001 C CNN
-F 3 "" H 1800 4100 50  0001 C CNN
-	1    1800 4100
-	1    0    0    -1
-$EndComp
-Wire Wire Line
-	1700 3700 1800 3700
-Wire Wire Line
-	1800 3700 1800 4100
-Text Label 3150 3950 2    60   ~ 0
+P 1300 3200
+F 0 "#PWR0133" H 1300 2950 50  0001 C CNN
+F 1 "GND" H 1305 3027 50  0000 C CNN
+F 2 "" H 1300 3200 50  0001 C CNN
+F 3 "" H 1300 3200 50  0001 C CNN
+	1    1300 3200
+	1    0    0    -1
+$EndComp
+Wire Wire Line
+	1200 2800 1300 2800
+Wire Wire Line
+	1300 2800 1300 3200
+Text Label 2650 3050 2    60   ~ 0
 2
 Wire Wire Line
-	2800 4050 3150 4050
-Wire Wire Line
-	2800 3950 3150 3950
-Wire Wire Line
-	2800 3850 3150 3850
-Text Label 3150 4050 2    60   ~ 0
+	2300 3150 2650 3150
+Wire Wire Line
+	2300 3050 2650 3050
+Wire Wire Line
+	2300 2950 2650 2950
+Text Label 2650 3150 2    60   ~ 0
 6(**)
-Text Label 3150 3850 2    60   ~ 0
+Text Label 2650 2950 2    60   ~ 0
 0(Rx)
 Wire Wire Line
@@
 3(**)
 Wire Wire Line
-	4100 3550 4400 3550
-Wire Wire Line
-	4200 3750 4200 3500
+	3250 3650 3400 3650
 $Comp
 L power:+5V #PWR0102
 U 1 1 5E35CD15
-P 4200 3500
+P 2250 3800
 AR Path="/5E35CD15" Ref="#PWR0102"  Part="1"
 AR Path="/5E34E778/5E35CD15" Ref="#PWR?"  Part="1"
-F 0 "#PWR0102" H 4200 3350 50  0001 C CNN
-F 1 "+5V" H 4215 3673 50  0000 C CNN
-F 2 "" H 4200 3500 50  0001 C CNN
-F 3 "" H 4200 3500 50  0001 C CNN
-	1    4200 3500
-	1    0    0    -1
-$EndComp
-$Comp
-L mylib:Thermocouple_PCB TC1
+F 0 "#PWR0102" H 2250 3650 50  0001 C CNN
+F 1 "+5V" H 2265 3973 50  0000 C CNN
+F 2 "" H 2250 3800 50  0001 C CNN
+F 3 "" H 2250 3800 50  0001 C CNN
+	1    2250 3800
+	1    0    0    -1
+$EndComp
+$Comp
+L Encoder_check-rescue:Thermocouple_PCB-mylib TC1
 U 1 1 5E39D361
 P 3800 1500
@@
 $EndComp
 $Comp
-L mylib:M78AR05-1 U5
+L Encoder_check-rescue:M78AR05-1-mylib U5
 U 1 1 5E3F9C08
 P 2700 1550
@@
 	5000 1450 5300 1450
 Wire Wire Line
-	1700 3900 2150 3900
-Wire Wire Line
-	1700 4000 2150 4000
+	1200 3000 1650 3000
+Wire Wire Line
+	1200 3100 1650 3100
 $Comp
 L Mechanical:MountingHole H4
@@
 	1    0    0    -1
 $EndComp
-$Comp
-L Connector_Generic:Conn_01x06 J2
-U 1 1 5E64F1F4
-P 3900 2700
-AR Path="/5E64F1F4" Ref="J2"  Part="1"
-AR Path="/5E331390/5E64F1F4" Ref="J?"  Part="1"
-F 0 "J2" H 3900 2200 50  0000 C CNN
-F 1 "Conn_01x06" H 3900 2300 50  0000 C CNN
-F 2 "TerminalBlock_TE-Connectivity:TerminalBlock_TE_282834-6_1x06_P2.54mm_Horizontal" H 3900 2700 50  0001 C CNN
-F 3 "~" H 3900 2700 50  0001 C CNN
-	1    3900 2700
-	-1   0    0    -1
-$EndComp
 Wire Wire Line
 	4100 2900 4450 2900
@@
 P 8150 5200
 F 0 "R26" H 8220 5246 50  0000 L CNN
-F 1 "R" H 8220 5155 50  0000 L CNN
+F 1 "10k" H 8220 5155 50  0000 L CNN
 F 2 "Resistor_SMD:R_0603_1608Metric" V 8080 5200 50  0001 C CNN
 F 3 "~" H 8150 5200 50  0001 C CNN
@@
 Wire Wire Line
 	6900 5650 6900 5600
-$Comp
-L Connector_Generic:Conn_01x10 J1
-U 1 1 5E852E79
-P 3850 3950
-F 0 "J1" H 3768 4567 50  0000 C CNN
-F 1 "Conn_01x10" H 3768 4476 50  0000 C CNN
-F 2 "Connector_Multicomp:Multicomp_MC9A12-1034_2x05_P2.54mm_Vertical" H 3850 3950 50  0001 C CNN
-F 3 "~" H 3850 3950 50  0001 C CNN
-	1    3850 3950
-	-1   0    0    -1
-$EndComp
-NoConn ~ 4050 3850
-NoConn ~ 4050 3550
+NoConn ~ 2500 3950
 $Comp
 L Device:LED D10
@@
 P 2850 5700
 F 0 "R27" H 2920 5746 50  0000 L CNN
-F 1 "R" H 2920 5655 50  0000 L CNN
+F 1 "1k" H 2920 5655 50  0000 L CNN
 F 2 "Resistor_SMD:R_0603_1608Metric" V 2780 5700 50  0001 C CNN
 F 3 "~" H 2850 5700 50  0001 C CNN
@@
 P 8300 5650
 F 0 "D11" V 8339 5533 50  0000 R CNN
-F 1 "LED" V 8248 5533 50  0000 R CNN
+F 1 "LED_RED" V 8248 5533 50  0000 R CNN
 F 2 "LED_SMD:LED_0603_1608Metric" H 8300 5650 50  0001 C CNN
 F 3 "~" H 8300 5650 50  0001 C CNN
@@
 P 8300 6000
 F 0 "R28" H 8370 6046 50  0000 L CNN
-F 1 "R" H 8370 5955 50  0000 L CNN
+F 1 "1k" H 8370 5955 50  0000 L CNN
 F 2 "Resistor_SMD:R_0603_1608Metric" V 8230 6000 50  0001 C CNN
 F 3 "~" H 8300 6000 50  0001 C CNN
@@
 	-1   0    0    1
 $EndComp
+$Comp
+L Connector_Generic:Conn_02x05_Odd_Even J1
+U 1 1 5E5B0699
+P 2700 4150
+F 0 "J1" H 2750 4567 50  0000 C CNN
+F 1 "Conn_02x05_Odd_Even" H 2750 4476 50  0000 C CNN
+F 2 "Connector_Multicomp:Multicomp_MC9A12-1034_2x05_P2.54mm_Vertical" H 2700 4150 50  0001 C CNN
+F 3 "~" H 2700 4150 50  0001 C CNN
+	1    2700 4150
+	1    0    0    -1
+$EndComp
+Wire Wire Line
+	2250 3800 2250 4050
+Wire Wire Line
+	2250 4050 2500 4050
+Wire Wire Line
+	3000 3950 3250 3950
+Wire Wire Line
+	3250 3650 3250 3950
+Wire Wire Line
+	3300 3950 3300 4550
+Wire Wire Line
+	3300 4550 2400 4550
+Wire Wire Line
+	2400 4550 2400 4150
+Wire Wire Line
+	2400 4150 2500 4150
+Wire Wire Line
+	3300 3950 4600 3950
+Wire Wire Line
+	3400 4150 3400 4650
+Wire Wire Line
+	3400 4650 2300 4650
+Wire Wire Line
+	2300 4650 2300 4250
+Wire Wire Line
+	2300 4250 2500 4250
+Wire Wire Line
+	3400 4150 4600 4150
+Wire Wire Line
+	3500 4350 3500 4750
+Wire Wire Line
+	3500 4750 2200 4750
+Wire Wire Line
+	2200 4750 2200 4350
+Wire Wire Line
+	2200 4350 2500 4350
+Wire Wire Line
+	3500 4350 4600 4350
+Wire Wire Line
+	3150 4450 3150 4350
+Wire Wire Line
+	3150 4350 3000 4350
+NoConn ~ 3000 4050
+Wire Wire Line
+	3150 4450 4600 4450
+Wire Wire Line
+	3000 4250 4600 4250
+Wire Wire Line
+	4600 4050 3150 4050
+Wire Wire Line
+	3150 4050 3150 4150
+Wire Wire Line
+	3150 4150 3000 4150
+$Comp
+L Connector:Screw_Terminal_01x06 J2
+U 1 1 5E88F264
+P 3900 2700
+F 0 "J2" H 3818 3117 50  0000 C CNN
+F 1 "Screw_Terminal_01x06" H 3818 3026 50  0000 C CNN
+F 2 "TerminalBlock_TE-Connectivity:TerminalBlock_TE_282834-6_1x06_P2.54mm_Horizontal" H 3900 2700 50  0001 C CNN
+F 3 "~" H 3900 2700 50  0001 C CNN
+	1    3900 2700
+	-1   0    0    -1
+$EndComp
 $EndSCHEMATC
