File: brake.sch (KiCad schematic (older format))
At the start: 10 parts, among them U6 INA180A, U7 A4953_LJ

Commit message: SPIにつなぐデバイスの電圧が違ったため設計ミスが判明。 これを修正した
Parts:
- U6: symbol mylib:INA180A -> Encoder_check-rescue:INA180A-mylib
Changed lines of the file:
@@
 EESchema Schematic File Version 4
-LIBS:Encoder_check-cache
 EELAYER 30 0
 EELAYER END
@@
 $EndDescr
 $Comp
-L mylib:INA180A U6
+L Encoder_check-rescue:INA180A-mylib U6
 U 1 1 5E529C75
 P 5250 4300
+AR Path="/5E529C75" Ref="U6"  Part="1"
+AR Path="/5E527F61/5E529C75" Ref="U6"  Part="1"
 F 0 "U6" H 5594 4346 50  0000 L CNN
 F 1 "INA180A" H 5450 4250 50  0000 L CNN
