File: rs485.sch (KiCad schematic (older format))
At the start: 4 parts, among them J5 Conn_01x02, U4 SP3481CN

Commit message: SPIにつなぐデバイスの電圧が違ったため設計ミスが判明。 これを修正した
Parts:
- R16: value R -> 120
Changed lines of the file:
@@
 EESchema Schematic File Version 4
-LIBS:Encoder_check-cache
 EELAYER 30 0
 EELAYER END
@@
 P 5050 3700
 F 0 "R16" H 5120 3746 50  0000 L CNN
-F 1 "R" H 5120 3655 50  0000 L CNN
+F 1 "120" H 5120 3655 50  0000 L CNN
 F 2 "Resistor_SMD:R_0603_1608Metric" V 4980 3700 50  0001 C CNN
 F 3 "~" H 5050 3700 50  0001 C CNN
