File: thermocouple.sch (KiCad schematic (older format))
At the start: 8 parts, among them U1 MAX31855KASA

Commit message: SPIにつなぐデバイスの電圧が違ったため設計ミスが判明。 これを修正した
Parts:
- C8: value C -> 0.1u
Changed lines of the file:
@@
 EESchema Schematic File Version 4
-LIBS:Encoder_check-cache
 EELAYER 30 0
 EELAYER END
@@
 P 6100 3000
 F 0 "C8" H 6215 3046 50  0000 L CNN
-F 1 "C" H 6215 2955 50  0000 L CNN
+F 1 "0.1u" H 6215 2955 50  0000 L CNN
 F 2 "Capacitor_SMD:C_0603_1608Metric" H 6138 2850 50  0001 C CNN
 F 3 "~" H 6100 3000 50  0001 C CNN
